File: Kicad9_Project/Power.kicad_sch (KiCad schematic)
At the start: 18 parts, among them U1 TP4056-42-ESOP8, U2 AMS1117-3.3

Commit message: kicad schematic update
Parts:
- C1, C2: footprint (none) -> Capacitor_SMD:C_0603_1608Metric
- C3, C4: footprint (none) -> Capacitor_SMD:C_Elec_5x5.4
- D1, D2, D3: footprint (none) -> LED_SMD:LED_1206_3216Metric
- R1, R2, R23, R3, R4, R5, R6: footprint (none) -> Resistor_SMD:R_0603_1608Metric
- RPROG1: renamed from RPROG; footprint (none) -> Resistor_SMD:R_0603_1608Metric
Changed lines of the file:
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@@
 			)
 		)
-		(property "Footprint" ""
+		(property "Footprint" "Capacitor_SMD:C_Elec_5x5.4"
 			(at 210.5152 68.58 0)
 			(effects
@@
 		(on_board yes)
 		(dnp no)
-		(property "Reference" "RPROG"
+		(property "Reference" "RPROG1"
 			(at 127 77.4699 0)
 			(effects
@@
 			)
 		)
-		(property "Footprint" ""
+		(property "Footprint" "Resistor_SMD:R_0603_1608Metric"
 			(at 122.682 78.74 90)
 			(effects
@@
 			(project ""
 				(path "/f0c57335-1044-469b-b8e4-ad3058badde6/d75cd807-c6ce-48c0-93f0-b274e72060cb"
-					(reference "RPROG")
+					(reference "RPROG1")
 					(unit 1)
 				)
@@
 			)
 		)
-		(property "Footprint" ""
+		(property "Footprint" "Resistor_SMD:R_0603_1608Metric"
 			(at 224.282 76.2 90)
 			(effects
@@
 			)
 		)
-		(property "Footprint" ""
+		(property "Footprint" "Resistor_SMD:R_0603_1608Metric"
 			(at 93.98 71.882 90)
 			(effects
@@
 			)
 		)
-		(property "Footprint" ""
+		(property "Footprint" "Resistor_SMD:R_0603_1608Metric"
 			(at 128.27 60.198 90)
 			(effects
@@
 			)
 		)
-		(property "Footprint" ""
+		(property "Footprint" "Resistor_SMD:R_0603_1608Metric"
 			(at 98.552 50.8 90)
 			(effects
@@
 			)
 		)
-		(property "Footprint" ""
+		(property "Footprint" "LED_SMD:LED_1206_3216Metric"
 			(at 88.9 62.23 0)
 			(effects
@@
 			)
 		)
-		(property "Footprint" ""
+		(property "Footprint" "Capacitor_SMD:C_Elec_5x5.4"
 			(at 183.8452 68.58 0)
 			(effects
@@
 			)
 		)
-		(property "Footprint" ""
+		(property "Footprint" "Resistor_SMD:R_0603_1608Metric"
 			(at 93.98 69.342 90)
 			(effects
@@
 			)
 		)
-		(property "Footprint" ""
+		(property "Footprint" "Capacitor_SMD:C_0603_1608Metric"
 			(at 69.5452 66.04 0)
 			(effects
@@
 			)
 		)
-		(property "Footprint" ""
+		(property "Footprint" "LED_SMD:LED_1206_3216Metric"
 			(at 78.74 62.23 0)
 			(effects
@@
 			)
 		)
-		(property "Footprint" ""
+		(property "Footprint" "Capacitor_SMD:C_0603_1608Metric"
 			(at 144.4752 73.66 0)
 			(effects
@@
 			)
 		)
-		(property "Footprint" ""
+		(property "Footprint" "LED_SMD:LED_1206_3216Metric"
 			(at 226.06 66.04 0)
 			(effects
@@
 			)
 		)
-		(property "Footprint" ""
+		(property "Footprint" "Resistor_SMD:R_0603_1608Metric"
 			(at 108.712 50.8 90)
 			(effects
@@
 			)
 		)
-		(property "Footprint" ""
+		(property "Footprint" "Resistor_SMD:R_0603_1608Metric"
 			(at 132.842 78.74 90)
 			(effects

Commit message: kicad update
Parts:
- BAT1: footprint (none) -> Connector_JST:JST_PH_B3B-PH-SM4-TB_1x03-1MP_P2.00mm_Vertical
- C3: value 10uF -> 22uF; footprint Capacitor_SMD:C_Elec_5x5.4 -> Capacitor_Tantalum_SMD:CP_EIA-3216-10_Kemet-I_HandSolder
- C4: footprint Capacitor_SMD:C_Elec_5x5.4 -> Capacitor_Tantalum_SMD:CP_EIA-3216-10_Kemet-I_HandSolder
Connections:
- net GND: now also BAT1.3 (Bat-); no longer BAT1. (NTC)
- net at C1.1, C3.1, U1.5 (BAT)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: now also BAT1.1 (Bat+); no longer BAT1. (NTC)
- net at R5.2, R6.1, U1.1 (TEMP): now also BAT1.2 (NTC); no longer BAT1. (NTC)
Changed lines of the file:
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@@
 			)
 		)
-		(property "Footprint" "Capacitor_SMD:C_Elec_5x5.4"
+		(property "Footprint" "Capacitor_Tantalum_SMD:CP_EIA-3216-10_Kemet-I_HandSolder"
 			(at 210.5152 68.58 0)
 			(effects
@@
 			)
 		)
-		(property "Footprint" ""
+		(property "Footprint" "Connector_JST:JST_PH_B3B-PH-SM4-TB_1x03-1MP_P2.00mm_Vertical"
 			(at 154.94 59.69 0)
 			(effects
@@
 			)
 		)
-		(pin ""
-		)
-		(pin ""
-		)
-		(pin ""
+		(pin "2"
+		)
+		(pin "3"
+		)
+		(pin "1"
 		)
 		(instances
@@
 			)
 		)
-		(property "Value" "10uF"
+		(property "Value" "22uF"
 			(at 186.69 65.1509 0)
 			(effects
@@
 			)
 		)
-		(property "Footprint" "Capacitor_SMD:C_Elec_5x5.4"
+		(property "Footprint" "Capacitor_Tantalum_SMD:CP_EIA-3216-10_Kemet-I_HandSolder"
 			(at 183.8452 68.58 0)
 			(effects
